Commit message: do more things

File: 02-inverse-dynamics/2link-robot.urdf (robot description, URDF)
Before this commit: robot 2link_robot, 4 links, 3 joints
Links:
- link arm1: mass None -> 1; geometry collision box size=0.2 .05 .05; visual box size=0.2 .05 .05
- link arm2: mass None -> 1; geometry collision box size=0.2 .05 .05; visual box size=0.2 .05 .05
Joints:
- joint baseHinge: axis 0 0 1 -> 0 0 0.1
- joint ee_joint: origin xyz=0.2 0 0 rpy=0 0 0 -> xyz=0.1 0 0.0 rpy=0 0 0
- joint interArm: origin xyz=0.2 0 0 rpy=0 0 0 -> xyz=0.2 0 0.0 rpy=0 0 0
